File: RT_PA_1_TSMC180.kicad_pcb (KiCad board)
At the start: 2 copper layers, 13 parts, among them SW1 SW_DIP_x03, SW10 SW_DIP_x02, SW11 SW_DIP_x02, SW12 SW_DIP_x02, SW2 SW_DIP_x03, SW3 SW_DIP_x03, SW4 SW_DIP_x02, SW5 SW_DIP_x02, SW6 SW_DIP_x01, SW7 SW_DIP_x02, SW8 SW_DIP_x02, SW9 SW_DIP_x02, U1 PART1p68

Commit message: Import project from Fatima's archive
Signed-off-by: Alexis Jeandet <alexis.jeandet@member.fsf.org>

Signed-off-by: Fatima Mehrez <fatima.mehrez@lpp.polytechnique.fr>
Parts:
- added C1: 1u, Capacitor_SMD:C_0603_1608Metric, F.Cu at (237.5, 210.8)
- added C100: 1u, Capacitor_SMD:C_0603_1608Metric, F.Cu at (256.5, 146.1)
- added C101: 1u, Capacitor_SMD:C_0603_1608Metric, F.Cu at (251.5, 158.8)
- added C102: 1u, Capacitor_SMD:C_0603_1608Metric, F.Cu at (261.6, 141.0)
- added C11: 10n, Capacitor_SMD:C_0603_1608Metric, F.Cu at (242.1, 205.8)
- added C12: 10n, Capacitor_SMD:C_0603_1608Metric, F.Cu at (234.1, 208.3)
- added C13: 1u, Capacitor_SMD:C_0603_1608Metric, F.Cu at (229.5, 212.6)
- added C15: 10n, Capacitor_SMD:C_0603_1608Metric, F.Cu at (238.8, 203.3)
- added C17: 1u, Capacitor_SMD:C_0603_1608Metric, F.Cu at (242.8, 200.8)
- added C19: 10n, Capacitor_SMD:C_0603_1608Metric, F.Cu at (238.1, 205.8)
- added C2: 1u, Capacitor_SMD:C_0603_1608Metric, F.Cu at (230.1, 205.1)
- added C21: 1u, Capacitor_SMD:C_0603_1608Metric, F.Cu at (233.5, 210.8)
- added C22: 10n, Capacitor_SMD:C_0603_1608Metric, F.Cu at (238.1, 208.3)
- added C23: 10n, Capacitor_SMD:C_0603_1608Metric, F.Cu at (242.8, 203.3)
- added C25: 1u, Capacitor_SMD:C_0603_1608Metric, F.Cu at (233.5, 213.3)
- added C27: 10n, Capacitor_SMD:C_0603_1608Metric, F.Cu at (238.8, 198.3)
- added C3: 1u, Capacitor_SMD:C_0603_1608Metric, F.Cu at (225.5, 209.7)
- added C32: 10n, Capacitor_SMD:C_0603_1608Metric, F.Cu at (238.8, 195.8)
- added C4: 1u, Capacitor_SMD:C_0603_1608Metric, F.Cu at (234.8, 198.3)
- added C42: 10n, Capacitor_SMD:C_0603_1608Metric, F.Cu at (225.5, 212.2)
- added C5: 1u, Capacitor_SMD:C_0603_1608Metric, F.Cu at (234.8, 195.8)
- added C50: 1n, Capacitor_SMD:C_0603_1608Metric, F.Cu at (227.9, 232.3)
- added C51: 1n, Capacitor_SMD:C_0603_1608Metric, F.Cu at (232.5, 230.1)
- added C52: 10n, Capacitor_SMD:C_0603_1608Metric, F.Cu at (230.1, 207.6)
- added C57: 1n, Capacitor_SMD:C_0603_1608Metric, F.Cu at (227.9, 234.8)
- added C6: 1u, Capacitor_SMD:C_0603_1608Metric, F.Cu at (238.8, 200.8)
- added C62: 10n, Capacitor_SMD:C_0603_1608Metric, F.Cu at (234.8, 203.3)
- added C7: 1u, Capacitor_SMD:C_0603_1608Metric, F.Cu at (242.8, 198.3)
- added C72: 10n, Capacitor_SMD:C_0603_1608Metric, F.Cu at (242.8, 195.8)
- added C8: 1u, Capacitor_SMD:C_0603_1608Metric, F.Cu at (229.5, 210.1)
- added C82: 10n, Capacitor_SMD:C_0603_1608Metric, F.Cu at (234.8, 200.8)
- added C9: 1u, Capacitor_SMD:C_0603_1608Metric, F.Cu at (234.1, 205.8)
- added J1: Conn_Coaxial, Connector_Coaxial:SMB_Jack_Vertical, F.Cu at (174.1, 238.1)
- added J10: Conn_01x01, Connector_PinHeader_2.54mm:PinHeader_1x01_P2.54mm_Vertical, F.Cu at (211.8, 206.1)
- added J11: Conn_01x01, Connector_PinHeader_2.54mm:PinHeader_1x01_P2.54mm_Vertical, F.Cu at (216.5, 196.8)
- added J12: Conn_01x01, Connector_PinHeader_2.54mm:PinHeader_1x01_P2.54mm_Vertical, F.Cu at (211.8, 201.5)
- added J13: Conn_01x01, Connector_PinHeader_2.54mm:PinHeader_1x01_P2.54mm_Vertical, F.Cu at (216.5, 201.5)
- added J14: Conn_01x01_Female, Connector:Banana_Jack_2Pin, F.Cu at (92.7, 135.7)
- added J15: Conn_01x01_Female, Connector:Banana_Jack_2Pin, F.Cu at (107.1, 147.7)
- added J16: Conn_01x01, Connector_PinHeader_2.54mm:PinHeader_1x01_P2.54mm_Vertical, F.Cu at (190.7, 230.8)
- added J17: Conn_01x03, Connector_PinHeader_2.54mm:PinHeader_1x03_P2.54mm_Vertical, F.Cu at (240.0, 220.5)
- added J18: Conn_01x01, Connector_PinHeader_2.54mm:PinHeader_1x01_P2.54mm_Vertical, F.Cu at (190.7, 235.4)
- added J19: Conn_01x01, Connector_PinHeader_2.54mm:PinHeader_1x01_P2.54mm_Vertical, F.Cu at (195.4, 230.8)
- added J2: Conn_01x01, Connector_PinHeader_2.54mm:PinHeader_1x01_P2.54mm_Vertical, F.Cu at (190.7, 226.1)
- added J20: Conn_01x01, Connector_PinHeader_2.54mm:PinHeader_1x01_P2.54mm_Vertical, F.Cu at (225.8, 206.1)
- added J21: Conn_01x01, Connector_PinHeader_2.54mm:PinHeader_1x01_P2.54mm_Vertical, F.Cu at (221.1, 210.8)
- added J22: Conn_01x01, Connector_PinHeader_2.54mm:PinHeader_1x01_P2.54mm_Vertical, F.Cu at (230.4, 196.8)
- added J23: Conn_01x01, Connector_PinHeader_2.54mm:PinHeader_1x01_P2.54mm_Vertical, F.Cu at (230.4, 201.5)
- added J24: Conn_01x01, Connector_PinHeader_2.54mm:PinHeader_1x01_P2.54mm_Vertical, F.Cu at (221.1, 206.1)
- added J25: Conn_01x01, Connector_PinHeader_2.54mm:PinHeader_1x01_P2.54mm_Vertical, F.Cu at (211.8, 196.8)
- added J26: Conn_01x01, Connector_PinHeader_2.54mm:PinHeader_1x01_P2.54mm_Vertical, F.Cu at (211.8, 210.8)
- added J27: Conn_01x01, Connector_PinHeader_2.54mm:PinHeader_1x01_P2.54mm_Vertical, F.Cu at (254.0, 220.5)
- added J28: Conn_01x01, Connector_PinHeader_2.54mm:PinHeader_1x01_P2.54mm_Vertical, F.Cu at (249.3, 225.2)
- added J29: Conn_Coaxial, Connector_Coaxial:SMB_Jack_Vertical, F.Cu at (188.3, 208.8)
- added J3: Conn_Coaxial, Connector_Coaxial:SMB_Jack_Vertical, F.Cu at (183.6, 238.1)
- added J30: Conn_01x01, Connector_PinHeader_2.54mm:PinHeader_1x01_P2.54mm_Vertical, F.Cu at (221.1, 196.8)
- added J31: Conn_Coaxial, Connector_Coaxial:SMB_Jack_Vertical, F.Cu at (178.7, 208.8)
- added J32: Conn_01x01, Connector_PinHeader_2.54mm:PinHeader_1x01_P2.54mm_Vertical, F.Cu at (216.5, 206.1)
- added J33: Conn_Coaxial, Connector_Coaxial:SMB_Jack_Vertical, F.Cu at (169.2, 208.8)
- added J34: Conn_01x01, Connector_PinHeader_2.54mm:PinHeader_1x01_P2.54mm_Vertical, F.Cu at (221.1, 201.5)
- added J35: Conn_Coaxial, Connector_Coaxial:SMB_Jack_Vertical, F.Cu at (188.3, 199.3)
- added J36: Conn_01x01, Connector_PinHeader_2.54mm:PinHeader_1x01_P2.54mm_Vertical, F.Cu at (225.8, 196.8)
- added J37: Conn_Coaxial, Connector_Coaxial:SMB_Jack_Vertical, F.Cu at (178.7, 199.3)
- added J38: Conn_01x01, Connector_PinHeader_2.54mm:PinHeader_1x01_P2.54mm_Vertical, F.Cu at (216.5, 210.8)
- added J39: Conn_Coaxial, Connector_Coaxial:SMB_Jack_Vertical, F.Cu at (169.2, 199.3)
- added J4: Conn_01x01, Connector_PinHeader_2.54mm:PinHeader_1x01_P2.54mm_Vertical, F.Cu at (162.1, 245.2)
- added J40: Conn_01x01, Connector_PinHeader_2.54mm:PinHeader_1x01_P2.54mm_Vertical, F.Cu at (225.8, 201.5)
- added J41: Conn_Coaxial, Connector_Coaxial:SMB_Jack_Vertical, F.Cu at (197.8, 208.8)
- added J42: Conn_01x01, Connector_PinHeader_2.54mm:PinHeader_1x01_P2.54mm_Vertical, F.Cu at (180.7, 215.9)
- added J43: Conn_Coaxial, Connector_Coaxial:SMB_Jack_Vertical, F.Cu at (197.8, 199.3)
- added J44: Conn_01x01, Connector_PinHeader_2.54mm:PinHeader_1x01_P2.54mm_Vertical, F.Cu at (166.7, 215.9)
- added J45: Conn_01x01, Connector_PinHeader_2.54mm:PinHeader_1x01_P2.54mm_Vertical, F.Cu at (249.3, 220.5)
- added J46: Conn_01x01, Connector_PinHeader_2.54mm:PinHeader_1x01_P2.54mm_Vertical, F.Cu at (244.7, 220.5)
- added J47: Conn_01x01, Connector_PinHeader_2.54mm:PinHeader_1x01_P2.54mm_Vertical, F.Cu at (171.4, 215.9)
- added J48: Conn_01x01, Connector_PinHeader_2.54mm:PinHeader_1x01_P2.54mm_Vertical, F.Cu at (176.0, 215.9)
- added J49: Conn_01x04, Connector_PinHeader_2.54mm:PinHeader_1x04_P2.54mm_Vertical, F.Cu at (162.1, 209.1)
- added J5: Conn_Coaxial, Connector_Coaxial:SMB_Jack_Vertical, F.Cu at (183.6, 228.6)
- added J50: Conn_01x04, Connector_PinHeader_2.54mm:PinHeader_1x04_P2.54mm_Vertical, F.Cu at (162.1, 196.8)
- added J51: Conn_01x01, Connector_PinHeader_2.54mm:PinHeader_1x01_P2.54mm_Vertical, F.Cu at (199.3, 215.9)
- added J52: Conn_01x01, Connector_PinHeader_2.54mm:PinHeader_1x01_P2.54mm_Vertical, F.Cu at (194.6, 215.9)
- added J53: Conn_01x01, Connector_PinHeader_2.54mm:PinHeader_1x01_P2.54mm_Vertical, F.Cu at (190.0, 215.9)
- added J54: Conn_01x01, Connector_PinHeader_2.54mm:PinHeader_1x01_P2.54mm_Vertical, F.Cu at (185.3, 215.9)
- added J55: Conn_01x02, Connector_PinHeader_2.54mm:PinHeader_1x02_P2.54mm_Vertical, F.Cu at (223.6, 233.3)
- added J56: Conn_01x02, Connector_PinHeader_2.54mm:PinHeader_1x02_P2.54mm_Vertical, F.Cu at (228.2, 226.1)
- added J57: Conn_01x02, Connector_PinHeader_2.54mm:PinHeader_1x02_P2.54mm_Vertical, F.Cu at (218.9, 233.3)
- added J58: Conn_01x03, Connector_PinHeader_2.54mm:PinHeader_1x03_P2.54mm_Vertical, F.Cu at (209.6, 226.1)
- added J59: Conn_01x01, Connector_PinHeader_2.54mm:PinHeader_1x01_P2.54mm_Vertical, F.Cu at (209.6, 235.8)
- added J6: Conn_01x01, Connector_PinHeader_2.54mm:PinHeader_1x01_P2.54mm_Vertical, F.Cu at (176.0, 245.2)
- added J60: Conn_01x02, Connector_PinHeader_2.54mm:PinHeader_1x02_P2.54mm_Vertical, F.Cu at (223.6, 226.1)
- added J61: Conn_01x02, Connector_PinHeader_2.54mm:PinHeader_1x02_P2.54mm_Vertical, F.Cu at (218.9, 226.1)
- added J62: Conn_01x03, Connector_PinHeader_2.54mm:PinHeader_1x03_P2.54mm_Vertical, F.Cu at (214.2, 226.1)
- added J63: Conn_01x01, Connector_PinHeader_2.54mm:PinHeader_1x01_P2.54mm_Vertical, F.Cu at (244.7, 225.2)
- added J64: Conn_01x01, Connector_PinHeader_2.54mm:PinHeader_1x01_P2.54mm_Vertical, F.Cu at (166.7, 245.2)
- added J65: Conn_Coaxial, Connector_Coaxial:SMB_Jack_Vertical, F.Cu at (164.5, 228.6)
- added J66: Conn_01x01, Connector_PinHeader_2.54mm:PinHeader_1x01_P2.54mm_Vertical, F.Cu at (171.4, 245.2)
- added J67: Conn_Coaxial, Connector_Coaxial:SMB_Jack_Vertical, F.Cu at (164.5, 238.1)
- added J7: Conn_Coaxial, Connector_Coaxial:SMB_Jack_Vertical, F.Cu at (174.1, 228.6)
- added J8: Conn_01x01, Connector_PinHeader_2.54mm:PinHeader_1x01_P2.54mm_Vertical, F.Cu at (195.4, 226.1)
- added J9: Conn_01x01_Female, Connector:Banana_Jack_2Pin, F.Cu at (107.1, 123.6)
- added R1: 50, Resistor_SMD:R_0603_1608Metric, F.Cu at (232.5, 227.6)
- added R2: 5k, Resistor_SMD:R_0603_1608Metric, F.Cu at (232.5, 225.1)
- added R3: 50k, Resistor_SMD:R_0603_1608Metric, F.Cu at (213.9, 237.3)
- added R4: 20k, Resistor_SMD:R_0603_1608Metric, F.Cu at (213.9, 234.8)
- added R5: 50k, Resistor_SMD:R_0603_1608Metric, F.Cu at (258.3, 161.3)
- added R6: 50k, Resistor_SMD:R_0603_1608Metric, F.Cu at (271.8, 137.2)
- added R7: 50k, Resistor_SMD:R_0603_1608Metric, F.Cu at (264.6, 148.6)
- SW10: value SW_DIP_x02 -> SW_DIP_x03; footprint Button_Switch_THT:SW_DIP_SPSTx02_Slide_6.7x6.64mm_W7.62mm_P2.54mm_LowProfile -> Button_Switch_THT:SW_DIP_SPSTx03_Slide_6.7x9.18mm_W7.62mm_P2.54mm_LowProfile
- SW12: value SW_DIP_x02 -> SW_DIP_x04; footprint Button_Switch_THT:SW_DIP_SPSTx02_Slide_6.7x6.64mm_W7.62mm_P2.54mm_LowProfile -> Button_Switch_THT:SW_DIP_SPSTx04_Slide_6.7x11.72mm_W7.62mm_P2.54mm_LowProfile
- moved SW1 104.3 mm to (214.6, 124.5)
- moved U1 81.9 mm to (188.0, 133.3)
- moved SW9 76.8 mm to (190.5, 171.4), turned to 90 degrees
- moved SW8 60.7 mm to (124.4, 176.7)
- moved SW3 57.6 mm to (102.7, 173.4)
- moved SW11 52.5 mm to (135.3, 179.2)
- moved SW4 44.3 mm to (124.4, 162.5)
- moved SW5 44.3 mm to (113.6, 173.4)
- moved SW12 39.8 mm to (163.8, 101.6)
- moved SW7 35.3 mm to (135.3, 162.5)
- moved SW2 33.6 mm to (102.7, 162.5)
- moved SW6 33.2 mm to (124.4, 170.8)
- moved SW10 32.7 mm to (113.6, 162.5)
Connections:
- net /Configs/1V8 renamed /1V8_g
- net /Configs/gnd renamed Net-(R1-Pad1)
- SW1 pad 4: /Configs/VDD_O -> /VDD_O
- SW1 pad 5: /Configs/VDD_M -> /VDD_M
- SW1 pad 6: /Configs/VDD_diff -> /VDD_diff
- SW10 pad 1: Net-(R1-Pad1) (its old number) -> Net-(SW10-Pad1)
- SW10 pad 2: Net-(R1-Pad1) (its old number) -> Net-(SW10-Pad1)
- SW10 pad 3: Net-(J27-Pad1) -> Net-(SW10-Pad1)
- SW11 pad 3: /Configs/VoO -> /VoO
- SW11 pad 4: /Configs/VoM -> /VoM
- SW12 pad 1: Net-(J28-Pad2) -> /VIbias
- SW12 pad 2: Net-(J28-Pad2) -> /VIbias
- SW12 pad 3: /Configs/VoO -> /VIbias
- SW12 pad 4: /Configs/VoM -> /VIbias
- SW2 pad 4: /Configs/GND_O -> /Vi1O
- SW2 pad 5: /Configs/GND_M -> /Vi1m
- SW2 pad 6: /Configs/GND_diff -> /Configs/Vi2d
- SW3 pad 1: /Configs/VIbias -> /Configs/Vi2d
- SW3 pad 2: /Configs/VIbias -> /Vi1m
- SW3 pad 3: /Configs/VIbias -> /Vi1O
- SW3 pad 4: /Configs/VbiasM -> Net-(SW10-Pad1)
- SW3 pad 5: /Configs/VbiasDiff -> Net-(SW10-Pad1)
- SW3 pad 6: /Configs/VbiasO -> Net-(SW10-Pad1)
- SW4 pad 1: /Configs/Vo1d -> /Vo1d
- SW4 pad 2: /Configs/Vo1d -> /Vo1d
- SW4 pad 3: /Configs/Vi1O -> /Vi1O
- SW4 pad 4: /Configs/Vi1m -> /Vi1m
- SW5 pad 1: /Configs/Vo2d -> /Vo2d
- SW5 pad 2: /Configs/Vo2d -> /Vo2d
- SW5 pad 3: /Configs/Vi2O -> /Vi2O
- SW5 pad 4: /Configs/Vi2m -> /Vi2m
- SW6 pad 1: /Configs/VoOi -> /VoOi
- SW6 pad 2: /Configs/Vbi -> Vbi
- SW7 pad 1: /Configs/VoOii -> /VoOii
- SW7 pad 2: /Configs/VoOii -> /VoOii
- SW7 pad 3: /Configs/VoOi -> /VoOi
- SW7 pad 4: /Configs/VoO -> /VoO
- SW8 pad 3: /Configs/Vbi -> Vbi
- SW8 pad 4: /Configs/Vo2O -> /Vo2O
- SW9 pad 3: /Configs/Vo1O -> /Vo1O
- SW9 pad 4: /Configs/Vbi -> Vbi
- U1 pad 11: /GND_M -> GND
- U1 pad 12: /VDD_M -> /VDD_M_3
- U1 pad 16: /GND_diff -> GND
- U1 pad 17: /VDD_diff -> /VDD_diff_1
- U1 pad 19: /GND_diff -> GND
- U1 pad 20: /VDD_diff -> /VDD_diff_2
- U1 pad 22: /GND_diff -> GND
- U1 pad 23: /VDD_diff -> /VDD_diff_3
- U1 pad 25: /GND_diff -> GND
- U1 pad 26: /VDD_diff -> /VDD_diff_4
- U1 pad 28: /VDD_O -> /VDD_O_1
- U1 pad 29: /GND_O -> GND
- U1 pad 35: /Vbi -> Vbi
- U1 pad 41: /VDD_O -> /VDD_O_2
- U1 pad 42: /GND_O -> GND
- U1 pad 43: /VDD_diff -> /VDD_diff_5
- U1 pad 44: /GND_diff -> GND
- U1 pad 47: /GND_io -> GND
- U1 pad 49: /VDD_diff -> /VDD_diff_6
- U1 pad 50: /GND_diff -> GND
- U1 pad 54: /VDD_diff -> /VDD_diff_7
- U1 pad 55: /GND_diff -> GND
- U1 pad 59: /VDD_diff -> /VDD_diff_8
- U1 pad 60: /GND_diff -> GND
- U1 pad 63: /GND_M -> GND
- U1 pad 64: /VDD_M -> /VDD_M_2
- U1 pad 7: /GND_M -> GND
- U1 pad 8: /VDD_M -> /VDD_M_1

Commit message: Major changes in almost all project sheets
Parts:
- moved SW12 71.9 mm to (232.4, 80.0)
Connections:
- net Vbi renamed /Vbi
