File: RT_PA_1_TSMC180.kicad_pcb (KiCad board)
At the start: 2 copper layers, 13 parts, among them SW1 SW_DIP_x03, SW10 SW_DIP_x02, SW11 SW_DIP_x02, SW12 SW_DIP_x02, SW2 SW_DIP_x03, SW3 SW_DIP_x03, SW4 SW_DIP_x02, SW5 SW_DIP_x02, SW6 SW_DIP_x01, SW7 SW_DIP_x02, SW8 SW_DIP_x02, SW9 SW_DIP_x02, U1 PART1p68

Commit message: Major changes in almost all project sheets-2
Parts:
- added C1: 1u, Capacitor_SMD:C_0603_1608Metric, F.Cu at (237.5, 210.8)
- added C100: 1u, Capacitor_SMD:C_0603_1608Metric, F.Cu at (256.5, 146.1)
- added C101: 1u, Capacitor_SMD:C_0603_1608Metric, F.Cu at (251.5, 158.8)
- added C102: 1u, Capacitor_SMD:C_0603_1608Metric, F.Cu at (261.6, 141.0)
- added C11: 10n, Capacitor_SMD:C_0603_1608Metric, F.Cu at (242.1, 205.8)
- added C12: 10n, Capacitor_SMD:C_0603_1608Metric, F.Cu at (234.1, 208.3)
- added C13: 1u, Capacitor_SMD:C_0603_1608Metric, F.Cu at (229.5, 212.6)
- added C15: 10n, Capacitor_SMD:C_0603_1608Metric, F.Cu at (238.8, 203.3)
- added C17: 1u, Capacitor_SMD:C_0603_1608Metric, F.Cu at (242.8, 200.8)
- added C19: 10n, Capacitor_SMD:C_0603_1608Metric, F.Cu at (238.1, 205.8)
- added C2: 1u, Capacitor_SMD:C_0603_1608Metric, F.Cu at (230.1, 205.1)
- added C21: 1u, Capacitor_SMD:C_0603_1608Metric, F.Cu at (233.5, 210.8)
- added C22: 10n, Capacitor_SMD:C_0603_1608Metric, F.Cu at (238.1, 208.3)
- added C23: 10n, Capacitor_SMD:C_0603_1608Metric, F.Cu at (242.8, 203.3)
- added C25: 1u, Capacitor_SMD:C_0603_1608Metric, F.Cu at (233.5, 213.3)
- added C27: 10n, Capacitor_SMD:C_0603_1608Metric, F.Cu at (238.8, 198.3)
- added C3: 1u, Capacitor_SMD:C_0603_1608Metric, F.Cu at (225.5, 209.7)
- added C32: 10n, Capacitor_SMD:C_0603_1608Metric, F.Cu at (238.8, 195.8)
- added C4: 1u, Capacitor_SMD:C_0603_1608Metric, F.Cu at (234.8, 198.3)
- added C42: 10n, Capacitor_SMD:C_0603_1608Metric, F.Cu at (225.5, 212.2)
- added C5: 1u, Capacitor_SMD:C_0603_1608Metric, F.Cu at (234.8, 195.8)
- added C50: 1n, Capacitor_SMD:C_0603_1608Metric, F.Cu at (227.9, 232.3)
- added C51: 1n, Capacitor_SMD:C_0603_1608Metric, F.Cu at (232.5, 230.1)
- added C52: 10n, Capacitor_SMD:C_0603_1608Metric, F.Cu at (230.1, 207.6)
- added C57: 1n, Capacitor_SMD:C_0603_1608Metric, F.Cu at (227.9, 234.8)
- added C6: 1u, Capacitor_SMD:C_0603_1608Metric, F.Cu at (238.8, 200.8)
- added C62: 10n, Capacitor_SMD:C_0603_1608Metric, F.Cu at (234.8, 203.3)
- added C7: 1u, Capacitor_SMD:C_0603_1608Metric, F.Cu at (242.8, 198.3)
- added C72: 10n, Capacitor_SMD:C_0603_1608Metric, F.Cu at (242.8, 195.8)
- added C8: 1u, Capacitor_SMD:C_0603_1608Metric, F.Cu at (229.5, 210.1)
- added C82: 10n, Capacitor_SMD:C_0603_1608Metric, F.Cu at (234.8, 200.8)
- added C9: 1u, Capacitor_SMD:C_0603_1608Metric, F.Cu at (234.1, 205.8)
- added J1: Conn_Coaxial, Connector_Coaxial:SMB_Jack_Vertical, F.Cu at (174.1, 238.1)
- added J10: Conn_01x01, Connector_PinHeader_2.54mm:PinHeader_1x01_P2.54mm_Vertical, F.Cu at (211.8, 206.1)
- added J11: Conn_01x01, Connector_PinHeader_2.54mm:PinHeader_1x01_P2.54mm_Vertical, F.Cu at (216.5, 196.8)
- added J12: Conn_01x01, Connector_PinHeader_2.54mm:PinHeader_1x01_P2.54mm_Vertical, F.Cu at (211.8, 201.5)
- added J13: Conn_01x01, Connector_PinHeader_2.54mm:PinHeader_1x01_P2.54mm_Vertical, F.Cu at (216.5, 201.5)
- added J14: Conn_01x01_Female, Connector:Banana_Jack_2Pin, F.Cu at (92.7, 135.7)
- added J15: Conn_01x01_Female, Connector:Banana_Jack_2Pin, F.Cu at (107.1, 147.7)
- added J16: Conn_01x01, Connector_PinHeader_2.54mm:PinHeader_1x01_P2.54mm_Vertical, F.Cu at (190.7, 230.8)
- added J17: Conn_01x03, Connector_PinHeader_2.54mm:PinHeader_1x03_P2.54mm_Vertical, F.Cu at (240.0, 220.5)
- added J18: Conn_01x01, Connector_PinHeader_2.54mm:PinHeader_1x01_P2.54mm_Vertical, F.Cu at (190.7, 235.4)
- added J19: Conn_01x01, Connector_PinHeader_2.54mm:PinHeader_1x01_P2.54mm_Vertical, F.Cu at (195.4, 230.8)
- added J2: Conn_01x01, Connector_PinHeader_2.54mm:PinHeader_1x01_P2.54mm_Vertical, F.Cu at (190.7, 226.1)
- added J20: Conn_01x01, Connector_PinHeader_2.54mm:PinHeader_1x01_P2.54mm_Vertical, F.Cu at (225.8, 206.1)
- added J21: Conn_01x01, Connector_PinHeader_2.54mm:PinHeader_1x01_P2.54mm_Vertical, F.Cu at (221.1, 210.8)
- added J22: Conn_01x01, Connector_PinHeader_2.54mm:PinHeader_1x01_P2.54mm_Vertical, F.Cu at (230.4, 196.8)
- added J23: Conn_01x01, Connector_PinHeader_2.54mm:PinHeader_1x01_P2.54mm_Vertical, F.Cu at (230.4, 201.5)
- added J24: Conn_01x01, Connector_PinHeader_2.54mm:PinHeader_1x01_P2.54mm_Vertical, F.Cu at (221.1, 206.1)
- added J25: Conn_01x01, Connector_PinHeader_2.54mm:PinHeader_1x01_P2.54mm_Vertical, F.Cu at (211.8, 196.8)
- added J26: Conn_01x01, Connector_PinHeader_2.54mm:PinHeader_1x01_P2.54mm_Vertical, F.Cu at (211.8, 210.8)
- added J27: Conn_01x01, Connector_PinHeader_2.54mm:PinHeader_1x01_P2.54mm_Vertical, F.Cu at (254.0, 220.5)
- added J28: Conn_01x01, Connector_PinHeader_2.54mm:PinHeader_1x01_P2.54mm_Vertical, F.Cu at (249.3, 225.2)
- added J29: Conn_Coaxial, Connector_Coaxial:SMB_Jack_Vertical, F.Cu at (188.3, 208.8)
- added J3: Conn_Coaxial, Connector_Coaxial:SMB_Jack_Vertical, F.Cu at (183.6, 238.1)
- added J30: Conn_01x01, Connector_PinHeader_2.54mm:PinHeader_1x01_P2.54mm_Vertical, F.Cu at (221.1, 196.8)
- added J31: Conn_Coaxial, Connector_Coaxial:SMB_Jack_Vertical, F.Cu at (178.7, 208.8)
- added J32: Conn_01x01, Connector_PinHeader_2.54mm:PinHeader_1x01_P2.54mm_Vertical, F.Cu at (216.5, 206.1)
- added J33: Conn_Coaxial, Connector_Coaxial:SMB_Jack_Vertical, F.Cu at (169.2, 208.8)
- added J34: Conn_01x01, Connector_PinHeader_2.54mm:PinHeader_1x01_P2.54mm_Vertical, F.Cu at (221.1, 201.5)
- added J35: Conn_Coaxial, Connector_Coaxial:SMB_Jack_Vertical, F.Cu at (188.3, 199.3)
- added J36: Conn_01x01, Connector_PinHeader_2.54mm:PinHeader_1x01_P2.54mm_Vertical, F.Cu at (225.8, 196.8)
- added J37: Conn_Coaxial, Connector_Coaxial:SMB_Jack_Vertical, F.Cu at (178.7, 199.3)
- added J38: Conn_01x01, Connector_PinHeader_2.54mm:PinHeader_1x01_P2.54mm_Vertical, F.Cu at (216.5, 210.8)
- added J39: Conn_Coaxial, Connector_Coaxial:SMB_Jack_Vertical, F.Cu at (169.2, 199.3)
- added J4: Conn_01x01, Connector_PinHeader_2.54mm:PinHeader_1x01_P2.54mm_Vertical, F.Cu at (162.1, 245.2)
- added J40: Conn_01x01, Connector_PinHeader_2.54mm:PinHeader_1x01_P2.54mm_Vertical, F.Cu at (225.8, 201.5)
- added J41: Conn_Coaxial, Connector_Coaxial:SMB_Jack_Vertical, F.Cu at (197.8, 208.8)
- added J42: Conn_01x01, Connector_PinHeader_2.54mm:PinHeader_1x01_P2.54mm_Vertical, F.Cu at (180.7, 215.9)
- added J43: Conn_Coaxial, Connector_Coaxial:SMB_Jack_Vertical, F.Cu at (197.8, 199.3)
- added J44: Conn_01x01, Connector_PinHeader_2.54mm:PinHeader_1x01_P2.54mm_Vertical, F.Cu at (166.7, 215.9)
- added J45: Conn_01x01, Connector_PinHeader_2.54mm:PinHeader_1x01_P2.54mm_Vertical, F.Cu at (249.3, 220.5)
- added J46: Conn_01x01, Connector_PinHeader_2.54mm:PinHeader_1x01_P2.54mm_Vertical, F.Cu at (244.7, 220.5)
- added J47: Conn_01x01, Connector_PinHeader_2.54mm:PinHeader_1x01_P2.54mm_Vertical, F.Cu at (171.4, 215.9)
- added J48: Conn_01x01, Connector_PinHeader_2.54mm:PinHeader_1x01_P2.54mm_Vertical, F.Cu at (176.0, 215.9)
- added J49: Conn_01x04, Connector_PinHeader_2.54mm:PinHeader_1x04_P2.54mm_Vertical, F.Cu at (162.1, 209.1)
- added J5: Conn_Coaxial, Connector_Coaxial:SMB_Jack_Vertical, F.Cu at (183.6, 228.6)
- added J50: Conn_01x04, Connector_PinHeader_2.54mm:PinHeader_1x04_P2.54mm_Vertical, F.Cu at (162.1, 196.8)
- added J51: Conn_01x01, Connector_PinHeader_2.54mm:PinHeader_1x01_P2.54mm_Vertical, F.Cu at (199.3, 215.9)
- added J52: Conn_01x01, Connector_PinHeader_2.54mm:PinHeader_1x01_P2.54mm_Vertical, F.Cu at (194.6, 215.9)
- added J53: Conn_01x01, Connector_PinHeader_2.54mm:PinHeader_1x01_P2.54mm_Vertical, F.Cu at (190.0, 215.9)
- added J54: Conn_01x01, Connector_PinHeader_2.54mm:PinHeader_1x01_P2.54mm_Vertical, F.Cu at (185.3, 215.9)
- added J55: Conn_01x02, Connector_PinHeader_2.54mm:PinHeader_1x02_P2.54mm_Vertical, F.Cu at (223.6, 233.3)
- added J56: Conn_01x02, Connector_PinHeader_2.54mm:PinHeader_1x02_P2.54mm_Vertical, F.Cu at (228.2, 226.1)
- added J57: Conn_01x02, Connector_PinHeader_2.54mm:PinHeader_1x02_P2.54mm_Vertical, F.Cu at (218.9, 233.3)
- added J58: Conn_01x03, Connector_PinHeader_2.54mm:PinHeader_1x03_P2.54mm_Vertical, F.Cu at (209.6, 226.1)
- added J59: Conn_01x01, Connector_PinHeader_2.54mm:PinHeader_1x01_P2.54mm_Vertical, F.Cu at (209.6, 235.8)
- added J6: Conn_01x01, Connector_PinHeader_2.54mm:PinHeader_1x01_P2.54mm_Vertical, F.Cu at (176.0, 245.2)
- added J60: Conn_01x02, Connector_PinHeader_2.54mm:PinHeader_1x02_P2.54mm_Vertical, F.Cu at (223.6, 226.1)
- added J61: Conn_01x02, Connector_PinHeader_2.54mm:PinHeader_1x02_P2.54mm_Vertical, F.Cu at (218.9, 226.1)
- added J62: Conn_01x03, Connector_PinHeader_2.54mm:PinHeader_1x03_P2.54mm_Vertical, F.Cu at (214.2, 226.1)
- added J63: Conn_01x01, Connector_PinHeader_2.54mm:PinHeader_1x01_P2.54mm_Vertical, F.Cu at (244.7, 225.2)
- added J64: Conn_01x01, Connector_PinHeader_2.54mm:PinHeader_1x01_P2.54mm_Vertical, F.Cu at (166.7, 245.2)
- added J65: Conn_Coaxial, Connector_Coaxial:SMB_Jack_Vertical, F.Cu at (164.5, 228.6)
- added J66: Conn_01x01, Connector_PinHeader_2.54mm:PinHeader_1x01_P2.54mm_Vertical, F.Cu at (171.4, 245.2)
- added J67: Conn_Coaxial, Connector_Coaxial:SMB_Jack_Vertical, F.Cu at (164.5, 238.1)
- added J7: Conn_Coaxial, Connector_Coaxial:SMB_Jack_Vertical, F.Cu at (174.1, 228.6)
- added J8: Conn_01x01, Connector_PinHeader_2.54mm:PinHeader_1x01_P2.54mm_Vertical, F.Cu at (195.4, 226.1)
- added J9: Conn_01x01_Female, Connector:Banana_Jack_2Pin, F.Cu at (107.1, 123.6)
- added R1: 50, Resistor_SMD:R_0603_1608Metric, F.Cu at (232.5, 227.6)
- added R2: 5k, Resistor_SMD:R_0603_1608Metric, F.Cu at (232.5, 225.1)
- added R3: 50k, Resistor_SMD:R_0603_1608Metric, F.Cu at (213.9, 237.3)
- added R4: 20k, Resistor_SMD:R_0603_1608Metric, F.Cu at (213.9, 234.8)
- added R5: 50k, Resistor_SMD:R_0603_1608Metric, F.Cu at (258.3, 161.3)
- added R6: 50k, Resistor_SMD:R_0603_1608Metric, F.Cu at (271.8, 137.2)
- added R7: 50k, Resistor_SMD:R_0603_1608Metric, F.Cu at (264.6, 148.6)
- SW10: value SW_DIP_x02 -> SW_DIP_x03; footprint Button_Switch_THT:SW_DIP_SPSTx02_Slide_6.7x6.64mm_W7.62mm_P2.54mm_LowProfile -> Button_Switch_THT:SW_DIP_SPSTx03_Slide_6.7x9.18mm_W7.62mm_P2.54mm_LowProfile
- SW12: value SW_DIP_x02 -> SW_DIP_x04; footprint Button_Switch_THT:SW_DIP_SPSTx02_Slide_6.7x6.64mm_W7.62mm_P2.54mm_LowProfile -> Button_Switch_THT:SW_DIP_SPSTx04_Slide_6.7x11.72mm_W7.62mm_P2.54mm_LowProfile
- moved SW12 105.2 mm to (232.4, 80.0)
- moved SW1 104.3 mm to (214.6, 124.5)
- moved U1 81.9 mm to (188.0, 133.3)
- moved SW9 76.8 mm to (190.5, 171.4), turned to 90 degrees
- moved SW8 60.7 mm to (124.4, 176.7)
- moved SW3 57.6 mm to (102.7, 173.4)
- moved SW11 52.5 mm to (135.3, 179.2)
- moved SW4 44.3 mm to (124.4, 162.5)
- moved SW5 44.3 mm to (113.6, 173.4)
- moved SW7 35.3 mm to (135.3, 162.5)
- moved SW2 33.6 mm to (102.7, 162.5)
- moved SW6 33.2 mm to (124.4, 170.8)
- moved SW10 32.7 mm to (113.6, 162.5)
Connections:
- net /Configs/1V8 renamed /1V8_g
- net /Configs/gnd renamed Net-(R1-Pad1)
- SW1 pad 4: /Configs/VDD_O -> /VDD_O
- SW1 pad 5: /Configs/VDD_M -> /VDD_M
- SW1 pad 6: /Configs/VDD_diff -> /VDD_diff
- SW10 pad 1: Net-(R1-Pad1) (its old number) -> Net-(SW10-Pad1)
- SW10 pad 2: Net-(R1-Pad1) (its old number) -> Net-(SW10-Pad1)
- SW10 pad 3: Net-(J27-Pad1) -> Net-(SW10-Pad1)
- SW11 pad 3: /Configs/VoO -> /VoO
- SW11 pad 4: /Configs/VoM -> /VoM
- SW12 pad 1: Net-(J28-Pad2) -> /VIbias
- SW12 pad 2: Net-(J28-Pad2) -> /VIbias
- SW12 pad 3: /Configs/VoO -> /VIbias
- SW12 pad 4: /Configs/VoM -> /VIbias
- SW2 pad 4: /Configs/GND_O -> /Vi1O
- SW2 pad 5: /Configs/GND_M -> /Vi1m
- SW2 pad 6: /Configs/GND_diff -> /Configs/Vi2d
- SW3 pad 1: /Configs/VIbias -> /Configs/Vi2d
- SW3 pad 2: /Configs/VIbias -> /Vi1m
- SW3 pad 3: /Configs/VIbias -> /Vi1O
- SW3 pad 4: /Configs/VbiasM -> Net-(SW10-Pad1)
- SW3 pad 5: /Configs/VbiasDiff -> Net-(SW10-Pad1)
- SW3 pad 6: /Configs/VbiasO -> Net-(SW10-Pad1)
- SW4 pad 1: /Configs/Vo1d -> /Vo1d
- SW4 pad 2: /Configs/Vo1d -> /Vo1d
- SW4 pad 3: /Configs/Vi1O -> /Vi1O
- SW4 pad 4: /Configs/Vi1m -> /Vi1m
- SW5 pad 1: /Configs/Vo2d -> /Vo2d
- SW5 pad 2: /Configs/Vo2d -> /Vo2d
- SW5 pad 3: /Configs/Vi2O -> /Vi2O
- SW5 pad 4: /Configs/Vi2m -> /Vi2m
- SW6 pad 1: /Configs/VoOi -> /VoOi
- SW6 pad 2: /Configs/Vbi -> /Vbi
- SW7 pad 1: /Configs/VoOii -> /VoOii
- SW7 pad 2: /Configs/VoOii -> /VoOii
- SW7 pad 3: /Configs/VoOi -> /VoOi
- SW7 pad 4: /Configs/VoO -> /VoO
- SW8 pad 3: /Configs/Vbi -> /Vbi
- SW8 pad 4: /Configs/Vo2O -> /Vo2O
- SW9 pad 3: /Configs/Vo1O -> /Vo1O
- SW9 pad 4: /Configs/Vbi -> /Vbi
- U1 pad 11: /GND_M -> GND
- U1 pad 12: /VDD_M -> /VDD_M_3
- U1 pad 16: /GND_diff -> GND
- U1 pad 17: /VDD_diff -> /VDD_diff_1
- U1 pad 19: /GND_diff -> GND
- U1 pad 20: /VDD_diff -> /VDD_diff_2
- U1 pad 22: /GND_diff -> GND
- U1 pad 23: /VDD_diff -> /VDD_diff_3
- U1 pad 25: /GND_diff -> GND
- U1 pad 26: /VDD_diff -> /VDD_diff_4
- U1 pad 28: /VDD_O -> /VDD_O_1
- U1 pad 29: /GND_O -> GND
- U1 pad 41: /VDD_O -> /VDD_O_2
- U1 pad 42: /GND_O -> GND
- U1 pad 43: /VDD_diff -> /VDD_diff_5
- U1 pad 44: /GND_diff -> GND
- U1 pad 47: /GND_io -> GND
- U1 pad 49: /VDD_diff -> /VDD_diff_6
- U1 pad 50: /GND_diff -> GND
- U1 pad 54: /VDD_diff -> /VDD_diff_7
- U1 pad 55: /GND_diff -> GND
- U1 pad 59: /VDD_diff -> /VDD_diff_8
- U1 pad 60: /GND_diff -> GND
- U1 pad 63: /GND_M -> GND
- U1 pad 64: /VDD_M -> /VDD_M_2
- U1 pad 7: /GND_M -> GND
- U1 pad 8: /VDD_M -> /VDD_M_1

Commit message: Adds missing Bias schematic, changes few footprints and started components grouping in PCB
Signed-off-by: Alexis Jeandet <alexis.jeandet@member.fsf.org>
Parts:
- added SW13: SW_DIP_x04, Button_Switch_THT:SW_DIP_SPSTx04_Slide_6.7x11.72mm_W7.62mm_P2.54mm_LowProfile, F.Cu at (387.0, 90.7)
- added SW14: SW_DIP_x04, Button_Switch_THT:SW_DIP_SPSTx04_Slide_6.7x11.72mm_W7.62mm_P2.54mm_LowProfile, F.Cu at (386.6, 138.6)
- added SW15: SW_DIP_x04, Button_Switch_THT:SW_DIP_SPSTx04_Slide_6.7x11.72mm_W7.62mm_P2.54mm_LowProfile, F.Cu at (386.5, 112.3)
- C1, C100, C101, C102, C13, C17, C2, C21, C25, C3, C4, C5, C6, C7, C8, C9: footprint Capacitor_SMD:C_0603_1608Metric -> Capacitor_SMD:C_0805_2012Metric_Pad1.18x1.45mm_HandSolder
- C11, C12, C15, C19, C22, C23, C27, C32, C42, C50, C51, C52, C57, C62, C72, C82: footprint Capacitor_SMD:C_0603_1608Metric -> Capacitor_SMD:C_0603_1608Metric_Pad1.08x0.95mm_HandSolder
- moved R1 233.2 mm to (12.7, 149.8)
- moved R2 192.1 mm to (57.7, 145.4)
- moved R3 178.9 mm to (58.0, 149.6)
- moved R4 175.4 mm to (58.2, 154.2)
- moved C8 150.2 mm to (379.7, 211.0)
- moved SW9 149.0 mm to (99.4, 289.4)
- moved C50 148.5 mm to (97.9, 160.5)
- moved C82 145.3 mm to (379.8, 208.9)
- moved R5 142.5 mm to (381.6, 89.9)
- moved C42 142.0 mm to (360.3, 256.7)
- moved C57 140.5 mm to (100.9, 295.0)
- moved C4 139.3 mm to (360.3, 258.7)
- moved C3 138.9 mm to (360.0, 244.1)
- moved C2 132.0 mm to (360.3, 226.8)
- moved C100 131.5 mm to (378.3, 96.5)
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Connections:
- J14 pad 2: (no net) -> /0V9_g
- J15 pad 2: (no net) -> /1V14_g
- J9 pad 2: (no net) -> /1V8_g

Commit message: Simplified VDD schematic nets
Signed-off-by: Alexis Jeandet <alexis.jeandet@member.fsf.org>
Connections:
- U1 pad 12: /VDD_M_3 -> /VDD_M
- U1 pad 17: /VDD_diff_1 -> /VDD_diff
- U1 pad 20: /VDD_diff_2 -> /VDD_diff
- U1 pad 23: /VDD_diff_3 -> /VDD_diff
- U1 pad 26: /VDD_diff_4 -> /VDD_diff
- U1 pad 28: /VDD_O_1 -> /VDD_O
- U1 pad 41: /VDD_O_2 -> /VDD_O
- U1 pad 43: /VDD_diff_5 -> /VDD_diff
- U1 pad 49: /VDD_diff_6 -> /VDD_diff
- U1 pad 54: /VDD_diff_7 -> /VDD_diff
- U1 pad 59: /VDD_diff_8 -> /VDD_diff
- U1 pad 64: /VDD_M_2 -> /VDD_M
- U1 pad 8: /VDD_M_1 -> /VDD_M

Commit message: Adds some missing connections and layout WIP
Signed-off-by: Alexis Jeandet <alexis.jeandet@member.fsf.org>
Parts:
- removed C1, C2, C3, C4, C5, C6, C7, C8: 1u, Capacitor_SMD:C_0805_2012Metric_Pad1.18x1.45mm_HandSolder
- removed J1, J29, J3, J31, J35, J41, J43, J5, J65, J67, J7: Conn_Coaxial, Connector_Coaxial:SMB_Jack_Vertical
- removed J10, J11, J12, J13, J16, J18, J19, J2, J27, J28, J30, J32, J34, J36, J38, J4, J40, J42, J44, J45, J46, J47, J48, J51, J52, J53, J54, J59, J6, J63, J64, J66, J8: Conn_01x01, Connector_PinHeader_2.54mm:PinHeader_1x01_P2.54mm_Vertical
- removed J17, J58, J62: Conn_01x03, Connector_PinHeader_2.54mm:PinHeader_1x03_P2.54mm_Vertical
- removed J49, J50: Conn_01x04, Connector_PinHeader_2.54mm:PinHeader_1x04_P2.54mm_Vertical
- removed J55, J56, J57, J60, J61: Conn_01x02, Connector_PinHeader_2.54mm:PinHeader_1x02_P2.54mm_Vertical
- added C201: 10uF, Capacitor_SMD:C_1206_3216Metric_Pad1.33x1.80mm_HandSolder, F.Cu at (193.2, 119.5)
- added C202: 10uF, Capacitor_SMD:C_1206_3216Metric_Pad1.33x1.80mm_HandSolder, F.Cu at (142.0, 124.5)
- C11, C12, C15, C19, C22, C23, C27, C32, C42, C50, C52, C62, C72, C82: moved to B.Cu
- moved C100 261.7 mm to (118.0, 123.0)
- moved R5 261.7 mm to (121.2, 116.4)
- moved SW13 261.7 mm to (126.6, 117.2)
- moved C82 242.3 mm to (152.7, 124.6), turned to 180 degrees
- moved C42 242.1 mm to (152.7, 132.2), turned to 180 degrees
- moved C32 229.4 mm to (161.4, 127.1)
- moved C9 219.2 mm to (160.7, 104.6)
- moved C17 214.8 mm to (177.5, 104.3)
- moved C13 213.4 mm to (150.1, 113.4), turned to 90 degrees
- moved C11 211.7 mm to (161.7, 114.0)
- moved C15 211.5 mm to (152.9, 114.4), turned to 180 degrees
- moved C25 210.4 mm to (150.6, 135.4), turned to 270 degrees
- moved C19 209.3 mm to (175.1, 113.8), turned to 180 degrees
- moved C27 205.3 mm to (155.3, 134.4), turned to 180 degrees
- moved C23 203.7 mm to (176.0, 137.8), turned to 270 degrees
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Connections:
- SW13 pad 5: /Configs/Vi1d -> /Vi1d
- SW13 pad 6: /Configs/Vi1d -> /Vi1d
- SW13 pad 7: /Configs/Vi1d -> /Vi1d
- SW13 pad 8: /Configs/Vi1d -> /Vi1d
- SW2 pad 6: /Configs/Vi2d -> /Vi2d
- SW3 pad 1: /Configs/Vi2d -> /Vi2d
Routing:
- net /T_Cc: track 0.00 -> 5.42 mm
- net /Vo2m: track 0.00 -> 2.64 mm

Commit message: Banana footprint change, added 3D models and PCB still WIP
Signed-off-by: Alexis Jeandet <alexis.jeandet@member.fsf.org>
Parts:
- added C401: NC, Capacitor_SMD:C_0805_2012Metric_Pad1.18x1.45mm_HandSolder, F.Cu at (98.6, 48.0)
- added C402: NC, Capacitor_SMD:C_0805_2012Metric_Pad1.18x1.45mm_HandSolder, B.Cu at (133.7, 49.5)
- added J1: Conn_Coaxial, Connector_Coaxial:SMB_Jack_Vertical, F.Cu at (91.2, 106.3)
- added J17: Conn_01x03, Connector_PinHeader_2.54mm:PinHeader_1x03_P2.54mm_Vertical, F.Cu at (61.1, 77.1)
- added J29: Conn_Coaxial, Connector_Coaxial:SMB_Jack_Vertical, F.Cu at (238.1, 68.6)
- added J3: Conn_Coaxial, Connector_Coaxial:SMB_Jack_Vertical, F.Cu at (89.9, 83.6)
- added J31: Conn_Coaxial, Connector_Coaxial:SMB_Jack_Vertical, F.Cu at (238.0, 89.0)
- added J35: Conn_Coaxial, Connector_Coaxial:SMB_Jack_Vertical, F.Cu at (237.6, 80.4)
- added J401: Conn_01x02, Connector_PinHeader_2.54mm:PinHeader_1x02_P2.54mm_Vertical, F.Cu at (146.1, 120.1)
- added J41: Conn_Coaxial, Connector_Coaxial:SMB_Jack_Vertical, F.Cu at (237.0, 157.0)
- added J43: Conn_Coaxial, Connector_Coaxial:SMB_Jack_Vertical, F.Cu at (236.6, 146.4)
- added J49: Conn_01x04, Connector_PinHeader_2.54mm:PinHeader_1x04_P2.54mm_Vertical, F.Cu at (167.9, 95.4)
- added J5: Conn_Coaxial, Connector_Coaxial:SMB_Jack_Vertical, F.Cu at (90.9, 95.2)
- added J50: Conn_01x04, Connector_PinHeader_2.54mm:PinHeader_1x04_P2.54mm_Vertical, F.Cu at (188.6, 146.3)
- added J55: Conn_01x02, Connector_PinHeader_2.54mm:PinHeader_1x02_P2.54mm_Vertical, F.Cu at (188.4, 60.8)
- added J56: Conn_01x02, Connector_PinHeader_2.54mm:PinHeader_1x02_P2.54mm_Vertical, F.Cu at (188.4, 68.0)
- added J57: Conn_01x02, Connector_PinHeader_2.54mm:PinHeader_1x02_P2.54mm_Vertical, F.Cu at (193.1, 68.0)
- added J58: Conn_01x03, Connector_PinHeader_2.54mm:PinHeader_1x03_P2.54mm_Vertical, F.Cu at (144.5, 101.6)
- added J60: Conn_01x02, Connector_PinHeader_2.54mm:PinHeader_1x02_P2.54mm_Vertical, F.Cu at (166.1, 159.5)
- added J61: Conn_01x02, Connector_PinHeader_2.54mm:PinHeader_1x02_P2.54mm_Vertical, F.Cu at (163.6, 142.0)
- added J62: Conn_01x03, Connector_PinHeader_2.54mm:PinHeader_1x03_P2.54mm_Vertical, F.Cu at (137.7, 148.7)
- added J65: Conn_Coaxial, Connector_Coaxial:SMB_Jack_Vertical, F.Cu at (237.9, 97.9)
- added J67: Conn_Coaxial, Connector_Coaxial:SMB_Jack_Vertical, F.Cu at (237.7, 106.7)
- added J7: Conn_Coaxial, Connector_Coaxial:SMB_Jack_Vertical, F.Cu at (92.5, 160.0)
- C51, C57: moved to B.Cu
- J14, J15, J9: value Conn_01x01_Female -> Conn_01x02_Female; footprint Connector:Banana_Jack_2Pin -> banana:Banana_test_point_4mm
- moved SW5 198.4 mm to (194.1, 106.0), turned to 270 degrees
- moved SW4 175.9 mm to (194.2, 124.6), turned to 270 degrees
- moved J33 173.2 mm to (236.5, 116.0), turned to 90 degrees
- moved C57 171.6 mm to (169.7, 137.8), turned to 90 degrees
- moved J39 168.6 mm to (236.6, 136.8), turned to 90 degrees
- moved C51 162.6 mm to (163.3, 137.8), turned to 90 degrees
- moved J37 162.2 mm to (236.5, 126.4), turned to 90 degrees
- moved SW9 150.9 mm to (168.4, 155.2)
- moved SW8 140.1 mm to (158.9, 155.2)
- moved R4 133.6 mm to (142.7, 50.8), turned to 90 degrees
- moved SW11 133.4 mm to (153.2, 46.5)
- moved SW3 131.6 mm to (118.3, 46.1)
- moved SW10 131.6 mm to (129.8, 45.8)
- moved SW2 131.6 mm to (106.0, 46.0)
- moved R1 131.6 mm to (98.6, 50.1)
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Routing:
- net /VDD_diff: track 0.00 -> 34.4 mm
- net Net-(C51-Pad1): track 0.00 -> 20.5 mm
- net /Vbi: track 0.00 -> 19.8 mm
- net Net-(C57-Pad1): track 0.00 -> 18.9 mm
- net /VDD_O: track 0.00 -> 18.8 mm
- net /Vo2O: track 0.00 -> 16.2 mm
- net /Vo1O: track 0.00 -> 12.8 mm
- net /VDD_M: track 0.00 -> 10.1 mm
- net /TCc1: track 0.00 -> 5.25 mm
- net /TCc2: track 0.00 -> 2.19 mm
